Commit message: refresh

File: irb120_description/urdf/irb120_2fgripper.urdf (robot description, URDF)
Before this commit: robot abb_irb120_model, 24 links, 23 joints
Links:
- removed link base
- added link end_effect_point, mass 0.001; visual box size=0.01 0.01 0.01
- link base_link: geometry collision mesh filename=package://irb120_description/meshes/visual/base_link.stl; visual mesh filename=package://irb120_description/meshes/visual/base_link.stl
- link coupling_link: geometry collision mesh filename=package://robotiq_2f_85_description/meshes/visual/robotiq_g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; visual mesh filename=package://robotiq_2f_85_description/meshes/visual/robotiq_g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
- link gripper_support_link: geometry collision mesh filename=package://irb120_description/meshes/supports/support_grippe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; visual mesh filename=package://irb120_description/meshes/supports/support_grippe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
- link left_inner_finger: mass None -> 0.0104003125914103; geometry collision mesh filename=package://robotiq_2f_85_description/meshes/visual/robotiq_a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 scale=0.001 0.001 0.001; visual mesh filename=package://robotiq_2f_85_description/meshes/visual/robotiq_a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 scale=0.001 0.001 0.001
- link left_inner_finger_pad: geometry collision box size=0.022 0.00635 0.0375; visual box size=0.022 0.00635 0.0375
- link left_inner_knuckle: mass None -> 0.0271177346495152; geometry collision mesh filename=package://robotiq_2f_85_description/meshes/visual/robotiq_a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 scale=0.001 0.001 0.001; visual mesh filename=package://robotiq_2f_85_description/meshes/visual/robotiq_a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 scale=0.001 0.001 0.001
- link left_outer_finger: mass None -> 0.022614240507152; geometry collision mesh filename=package://robotiq_2f_85_description/meshes/visual/robotiq_a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 scale=0.001 0.001 0.001; visual mesh filename=package://robotiq_2f_85_description/meshes/visual/robotiq_a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 scale=0.001 0.001 0.001
- link left_outer_knuckle: mass None -> 0.00853198276973456; geometry collision mesh filename=package://robotiq_2f_85_description/meshes/visual/robotiq_a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 scale=0.001 0.001 0.001; visual mesh filename=package://robotiq_2f_85_description/meshes/visual/robotiq_a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 scale=0.001 0.001 0.001
- link link_1: geometry collision mesh filename=package://irb120_description/meshes/visual/link_1.stl; visual mesh filename=package://irb120_description/meshes/visual/link_1.stl
- link link_2: geometry collision mesh filename=package://irb120_description/meshes/visual/link_2.stl; visual mesh filename=package://irb120_description/meshes/visual/link_2.stl
- link link_3: geometry collision mesh filename=package://irb120_description/meshes/visual/link_3.stl; visual mesh filename=package://irb120_description/meshes/visual/link_3.stl
- link link_4: geometry collision mesh filename=package://irb120_description/meshes/visual/link_4.stl; visual mesh filename=package://irb120_description/meshes/visual/link_4.stl
- link link_5: geometry collision mesh filename=package://irb120_description/meshes/visual/link_5.stl; visual mesh filename=package://irb120_description/meshes/visual/link_5.stl
- link link_6: geometry collision mesh filename=package://irb120_description/meshes/visual/link_6.stl; visual mesh filename=package://irb120_description/meshes/visual/link_6.stl
- link right_inner_finger: mass None -> 0.0104003125914103; geometry collision mesh filename=package://robotiq_2f_85_description/meshes/visual/robotiq_a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 scale=0.001 0.001 0.001; visual mesh filename=package://robotiq_2f_85_description/meshes/visual/robotiq_a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 scale=0.001 0.001 0.001
- link right_inner_finger_pad: geometry collision box size=0.022 0.00635 0.0375; visual box size=0.022 0.00635 0.0375
- link right_inner_knuckle: mass None -> 0.0271177346495152; geometry collision mesh filename=package://robotiq_2f_85_description/meshes/visual/robotiq_a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 scale=0.001 0.001 0.001; visual mesh filename=package://robotiq_2f_85_description/meshes/visual/robotiq_a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 scale=0.001 0.001 0.001
- link right_outer_finger: mass None -> 0.022614240507152; geometry collision mesh filename=package://robotiq_2f_85_description/meshes/visual/robotiq_a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 scale=0.001 0.001 0.001; visual mesh filename=package://robotiq_2f_85_description/meshes/visual/robotiq_a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 scale=0.001 0.001 0.001
- link right_outer_knuckle: mass None -> 0.00853198276973456; geometry collision mesh filename=package://robotiq_2f_85_description/meshes/visual/robotiq_a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 scale=0.001 0.001 0.001; visual mesh filename=package://robotiq_2f_85_description/meshes/visual/robotiq_a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 scale=0.001 0.001 0.001
- link robotiq_arg2f_base_link: geometry collision mesh filename=package://robotiq_2f_85_description/meshes/visual/robotiq_a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; visual mesh filename=package://robotiq_2f_85_description/meshes/visual/robotiq_a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 scale=0.001 0.001 0.001
Joints:
- removed joint base_link-base
- added joint end_effect_point: type fixed, parent gripper_support_link, child end_effect_point, origin xyz=0 0 0.15 rpy=0 0 0
- joint joint_1: limit lower=-2.87979 upper=2.87979 effort=0 velocity=4.36332 -> lower=-2.87979 upper=2.87979 effort=30 velocity=4.36332
- joint joint_2: limit lower=-1.91986 upper=1.91986 effort=0 velocity=4.36332 -> lower=-1.91986 upper=1.91986 effort=30 velocity=4.36332
- joint joint_3: limit lower=-1.91986 upper=1.22173 effort=0 velocity=4.36332 -> lower=-1.91986 upper=1.22173 effort=30 velocity=4.36332
- joint joint_4: limit lower=-2.79253 upper=2.79253 effort=0 velocity=5.58505 -> lower=-2.79253 upper=2.79253 effort=30 velocity=5.58505
- joint joint_5: limit lower=-2.094395 upper=2.094395 effort=0 velocity=5.58505 -> lower=-2.094395 upper=2.094395 effort=30 velocity=5.58505
- joint joint_6: limit lower=-6.98132 upper=6.98132 effort=0 velocity=7.33038 -> lower=-6.98132 upper=6.98132 effort=30 velocity=7.33038
- joint left_inner_finger_joint: limit lower=0 upper=0.8757 effort=1000 velocity=2.0 -> lower=-0.8757 upper=0.8757 effort=1000 velocity=2.0
- joint right_inner_finger_joint: limit lower=0 upper=0.8757 effort=1000 velocity=2.0 -> lower=-0.8757 upper=0.8757 effort=1000 velocity=2.0

Commit message: update

File: irb120_description/urdf/irb120_2fgripper.urdf (robot description, URDF)
Before this commit: robot abb_irb120_model, 24 links, 23 joints
Links:
- removed link gripper_support_link
Joints:
- removed joint irb120_joint_gripper_support
- joint end_effect_point: parent gripper_support_link -> tool0
- joint irb120_support_gripper: parent gripper_support_link -> tool0
