Commit message: update

File: irb120_description/urdf/gripper_2f.xacro (robot description, xacro)
@@ -4,5 +4,5 @@
 	<xacro:property name="PI" value="3.1415926535897931"/>
  <!-- verificar angulo de support_gripper -->
-  <link name="gripper_support_link">
+  <!-- <link name="gripper_support_link">
     <inertial>
       <origin
@@ -38,19 +38,19 @@
       </geometry>
     </collision>
-  </link>
+  </link> -->
   <joint name="irb120_joint_gripper_support" type="fixed">
     <parent link="tool0"/>
-    <child link="gripper_support_link"/>
-    <origin rpy="0 0 0" xyz="0 0 0.008"/>
+    <child link="coupling_link"/>
+    <origin rpy="0 0 0" xyz="0 0 -0.003"/>
   </joint>
-  <joint name="irb120_support_gripper" type="fixed">
+  <!-- <joint name="irb120_support_gripper" type="fixed">
     <parent link="gripper_support_link"/>
     <child link="coupling_link"/>
     <origin rpy="0 0 0" xyz="0 0 0"/>
-  </joint>
+  </joint> -->
   <!-- end effect point -->
   <joint name="end_effect_point" type="fixed">
     <origin rpy="0 0 0" xyz="0 0 0.15"/>
-    <parent link="gripper_support_link"/>
+    <parent link="coupling_link"/>
     <child link="end_effect_point"/>
   </joint>
@@ -58,7 +58,7 @@
   <link name="end_effect_point">
     <visual>
-      <origin rpy="0 0 0" xyz="0 0 0"/>
+      <origin rpy="0 0 0" xyz="0 0 -0.1"/>
       <geometry>
-        <box size="0.01 0.01 0.01"/>
+        <box size="0.02 0.02 0.02"/>
       </geometry>
       <material name="">
@@ -66,9 +66,9 @@
       </material>
     </visual>
-    <inertial>
+    <!-- <inertial>
       <origin rpy="0 0 0" xyz="0.0 0.0 0.0"/>
       <mass value="0.001"/>
       <inertia ixx="1.0e-06" ixy="0.0" ixz="0.0" iyy="1.0e-06" iyz="0.0" izz="1.0e-06"/>
-    </inertial>
+    </inertial> -->
   </link>
 </robot>
