Commit message: refresh

File: irb120_description/urdf/irb120.xacro (robot description, xacro)
@@ -1,324 +1,226 @@
-<?xml version="1.0" ?>
-<robot name="irb120_ABB"
-    xmlns:xacro="http://ros.org/wiki/xacro">
-    <xacro:include filename="$(find irb120_description)/urdf/common_materials.xacro"/>
-    <!-- ros_control plugin -->
-    <gazebo>
-        <plugin name="gazebo_ros_control" filename="libgazebo_ros_control.so">
-            <robotNamespace>/</robotNamespace>
-            <robotSimType>gazebo_ros_control/DefaultRobotHWSim</robotSimType>
-        </plugin>
-    </gazebo>
-    <xacro:property name="irb120_ns" value="" />
-    <!-- Used for fixing robot to Gazebo 'base_link' -->
-    <link name="world"/>
-    <joint name="fixed" type="fixed">
-        <parent link="world"/>
-        <child link="${irb120_ns}base_link"/>
-        <origin rpy="0 0 0" xyz="0 0 0"/>
-    </joint>
-    <!-- Description of IRB120 robot -->
-    <!-- Description of base_link -->
-    <link name="${irb120_ns}base_link">
-        <inertial>
-            <mass value="6.215"/>
-            <origin xyz="0 0 0" rpy="0 0 0"/>
-            <inertia ixx="0.0247272" ixy="-8.0784E-05" ixz="0.00130902" iyy="0.0491285" iyz="-8.0419E-06" izz="0.0472376"/>
-        </inertial>
-        <visual>
-            <origin xyz="0 0 0" rpy="0 0 0"/>
-            <geometry>
-                <mesh filename="package://irb120_description/mesh/irb120/base_link.stl"/>
-            </geometry>
-            <xacro:material_abb_orange />
-        </visual>
-        <collision>
-            <origin xyz="0 0 0" rpy="0 0 0"/>
-            <geometry>
-                <mesh filename="package://irb120_description/collision/irb120/base_link.stl"/>
-            </geometry>
-            <xacro:material_abb_yellow />
-        </collision>
-    </link>
-    <!-- Joint - 1 -->
-    <joint name="${irb120_ns}joint_1" type="revolute">
-        <origin rpy="0 0 0" xyz="0 0 0"/>
-        <parent link="${irb120_ns}base_link"/>
-        <child link="${irb120_ns}link_1"/>
-        <limit effort="20" lower="-2.87979" upper="2.87979" velocity="4.36332"/>
-        <axis xyz="0 0 1"/>
-        <dynamics damping="1" friction="0"/>
-    </joint>
-    <!-- Description of link - 1 -->
-    <link name="${irb120_ns}link_1">
-        <inertial>
-            <mass value="3.067" />
-            <origin xyz="0 0 0.23841" rpy="0 0 0"/>
-            <inertia ixx="0.0142175" ixy="-1.28579E-05" ixz="-2.31364E-05" iyy="0.0144041" iyz="1.93404E-05" izz="0.0104533"/>
-        </inertial>
-        <visual>
-            <origin xyz="0 0 0" rpy="0 0 0"/>
-            <geometry>
-                <mesh filename="package://irb120_description/mesh/irb120/link_1.stl"/>
-            </geometry>
-            <xacro:material_abb_orange />
-        </visual>
-        <collision>
-            <origin xyz="0 0 0" rpy="0 0 0"/>
-            <geometry>
-                <mesh filename="package://irb120_description/collision/irb120/link_1.stl"/>
-            </geometry>
-            <xacro:material_abb_yellow />
-        </collision>
-    </link>
-    <!-- Joint - 2 -->
-    <joint name="${irb120_ns}joint_2" type="revolute">
-        <origin rpy="0 0 0" xyz="0 0 0.29"/>
-        <parent link="${irb120_ns}link_1"/>
-        <child link="${irb120_ns}link_2"/>
-        <limit effort="20" lower="-1.91986" upper="1.91986" velocity="4.36332"/>
-        <axis xyz="0 1 0"/>
-        <dynamics damping="1" friction="0"/>
-    </joint>
-    <!-- Description of link - 2 -->
-    <link name="${irb120_ns}link_2">
-        <inertial>
-            <mass value="3.909"/>
-            <origin xyz="0.00078 -0.00212 0.10124" rpy="0 0 0"/>
-            <inertia ixx="0.0603111" ixy="9.83431E-06" ixz="5.72407E-05" iyy="0.041569" iyz="-0.00050497" izz="0.0259548"/>
-        </inertial>
-        <visual>
-            <origin xyz="0 0 0" rpy="0 0 0"/>
-            <geometry>
-                <mesh filename="package://irb120_description/mesh/irb120/link_2.stl"/>
-            </geometry>
-            <xacro:material_abb_orange />
-        </visual>
-        <collision>
-            <origin xyz="0 0 0" rpy="0 0 0"/>
-            <geometry>
-                <mesh filename="package://irb120_description/collision/irb120/link_2.stl"/>
-            </geometry>
-            <xacro:material_abb_yellow />
-        </collision>
-    </link>
-    <!-- Joint - 3 -->
-    <joint name="${irb120_ns}joint_3" type="revolute">
-        <origin rpy="0 0 0" xyz="0 0 0.27"/>
-        <parent link="${irb120_ns}link_2"/>
-        <child link="${irb120_ns}link_3"/>
-        <limit effort="20" lower="-1.91986" upper="1.22173" velocity="4.36332"/>
-        <axis xyz="0 1 0"/>
-        <dynamics damping="1" friction="0.0"/>
-    </joint>
-    <!-- Description of link - 3 -->
-    <link name="${irb120_ns}link_3">
-        <inertial>
-            <mass value="2.944"/>
-            <origin xyz="0.02281 0.00106 0.05791" rpy="0 0 0"/>
-            <inertia ixx="0.00835606" ixy="-8.01545E-05" ixz="0.00142884" iyy="0.016713" iyz="-0.000182227" izz="0.0126984"/>
-        </inertial>
-        <visual>
-            <origin xyz="0 0 0" rpy="0 0 0"/>
-            <geometry>
-                <mesh filename="package://irb120_description/mesh/irb120/link_3.stl"/>
-            </geometry>
-            <xacro:material_abb_orange />
-        </visual>
-        <collision>
-            <origin xyz="0 0 0" rpy="0 0 0"/>
-            <geometry>
-                <mesh filename="package://irb120_description/collision/irb120/link_3.stl"/>
-            </geometry>
-            <xacro:material_abb_yellow />
-        </collision>
-    </link>
-    <!-- Joint - 4 -->
-    <joint name="${irb120_ns}joint_4" type="revolute">
-        <origin rpy="0 0 0" xyz="0 0 0.07"/>
-        <parent link="${irb120_ns}link_3"/>
-        <child link="${irb120_ns}link_4"/>
-        <limit effort="20" lower="-2.792526" upper="2.792526" velocity="5.58505"/>
-        <axis xyz="1 0 0"/>
-        <dynamics damping="1" friction="0"/>
-    </joint>
-    <!--  Description of link - 4 -->
-    <link name="${irb120_ns}link_4">
-        <inertial>
-            <mass value="0.1328"/>
-            <origin xyz="0.2247 0.00015 0.00041" rpy="0 0 0"/>
-            <inertia ixx="0.00284661" ixy="-2.12765E-05" ixz="-1.6435E-05" iyy="0.00401346" iyz="1.31336E-05" izz="0.0052535"/>
-        </inertial>
-        <visual>
-            <origin xyz="0 0 0" rpy="0 0 0"/>
-            <geometry>
-                <mesh filename="package://irb120_description/mesh/irb120/link_4.stl"/>
-            </geometry>
-            <xacro:material_abb_orange />
-        </visual>
-        <collision>
-            <origin xyz="0 0 0" rpy="0 0 0"/>
-            <geometry>
-                <mesh filename="package://irb120_description/collision/irb120/link_4.stl"/>
-            </geometry>
-            <xacro:material_abb_yellow />
-        </collision>
-    </link>
-    <!-- Joint - 5 -->
-    <joint name="${irb120_ns}joint_5" type="revolute">
-        <origin rpy="0 0 0" xyz="0.302 0 0"/>
-        <parent link="${irb120_ns}link_4"/>
-        <child link="${irb120_ns}link_5"/>
-        <limit effort="20" lower="-2.094395" upper="2.094395" velocity="5.58505"/>
-        <axis xyz="0 1 0"/>
-        <dynamics damping="1" friction="0.0"/>
-    </joint>
-    <!-- Description of link - 5-->
-    <link name="${irb120_ns}link_5">
-        <inertial>
-            <mass value="0.546"/>
-            <origin xyz="-0.00109 3.68E-05 6.22E-05" rpy="0 0 0"/>
-            <inertia ixx="0.00284661" ixy="-2.12765E-05" ixz="-1.6435E-05" iyy="0.00401346" iyz="1.31336E-05" izz="0.0052535"/>
-        </inertial>
-        <visual>
-            <origin xyz="0 0 0" rpy="0 0 0"/>
-            <geometry>
-                <mesh filename="package://irb120_description/mesh/irb120/link_5.stl"/>
-            </geometry>
-            <xacro:material_abb_orange />
-        </visual>
-        <collision>
-            <origin xyz="0 0 0" rpy="0 0 0"/>
-            <geometry>
-                <mesh filename="package://irb120_description/collision/irb120/link_5.stl"/>
-            </geometry>
-            <xacro:material_abb_yellow />
-        </collision>
-    </link>
-    <!-- Joint - 6 -->
-    <joint name="${irb120_ns}joint_6" type="revolute">
-        <origin rpy="0 0 0" xyz="0.072 0 0"/>
-        <parent link="${irb120_ns}link_5"/>
-        <child link="${irb120_ns}link_6"/>
-        <limit effort="20" lower="-6.981317" upper="6.981317" velocity="7.33038"/>
-        <axis xyz="1 0 0"/>
-        <dynamics damping="1" friction="0.0"/>
-    </joint>
-    <!-- Description of link - 6 -->
-    <link name="${irb120_ns}link_6">
-        <inertial>
-            <mass value="0.137"/>
-            <origin xyz="-0.00706 -0.00017 -1.32E-06" rpy="0 0 0"/>
-            <inertia ixx="0.00284661" ixy="-2.12765E-05" ixz="-1.6435E-05" iyy="0.00401346" iyz="1.31336E-05" izz="0.0052535"/>
-        </inertial>
-        <visual>
-            <origin xyz="0 0 0" rpy="0 0 0"/>
-            <geometry>
-                <mesh filename="package://irb120_description/mesh/irb120/link_6.stl"/>
-            </geometry>
-            <xacro:material_abb_black />
-        </visual>
-        <collision>
-            <origin xyz="0 0 0" rpy="0 0 0"/>
-            <geometry>
-                <mesh filename="package://irb120_description/collision/irb120/link_6.stl"/>
-            </geometry>
-            <xacro:material_abb_yellow />
-        </collision>
-    </link>
-    <!-- Robot kinetics parts -->
-    <!-- transmission list -->
-    <transmission name="${irb120_ns}tran1">
-        <type>transmission_interface/SimpleTransmission</type>
-        <joint name="${irb120_ns}joint_1">
-            <hardwareInterface>PositionJointInterface</hardwareInterface>
-        </joint>
-        <actuator name="${irb120_ns}motor1">
-            <mechanicalReduction>1</mechanicalReduction>
-        </actuator>
-    </transmission>
-    <transmission name="${irb120_ns}tran2">
-        <type>transmission_interface/SimpleTransmission</type>
-        <joint name="${irb120_ns}joint_2">
-            <hardwareInterface>PositionJointInterface</hardwareInterface>
-        </joint>
-        <actuator name="${irb120_ns}motor2">
-            <mechanicalReduction>1</mechanicalReduction>
-        </actuator>
-    </transmission>
-    <transmission name="${irb120_ns}tran3">
-        <type>transmission_interface/SimpleTransmission</type>
-        <joint name="${irb120_ns}joint_3">
-            <hardwareInterface>PositionJointInterface</hardwareInterface>
-        </joint>
-        <actuator name="${irb120_ns}motor3">
-            <mechanicalReduction>1</mechanicalReduction>
-        </actuator>
-    </transmission>
-    <transmission name="${irb120_ns}tran4">
-        <type>transmission_interface/SimpleTransmission</type>
-        <joint name="${irb120_ns}joint_4">
-            <hardwareInterface>PositionJointInterface</hardwareInterface>
-        </joint>
-        <actuator name="${irb120_ns}motor4">
-            <mechanicalReduction>1</mechanicalReduction>
-        </actuator>
-    </transmission>
-    <transmission name="${irb120_ns}tran5">
-        <type>transmission_interface/SimpleTransmission</type>
-        <joint name="${irb120_ns}joint_5">
-            <hardwareInterface>PositionJointInterface</hardwareInterface>
-        </joint>
-        <actuator name="${irb120_ns}motor5">
-            <mechanicalReduction>1</mechanicalReduction>
-        </actuator>
-    </transmission>
-    <transmission name="${irb120_ns}tran6">
-        <type>transmission_interface/SimpleTransmission</type>
-        <joint name="${irb120_ns}joint_6">
-            <hardwareInterface>PositionJointInterface</hardwareInterface>
-        </joint>
-        <actuator name="${irb120_ns}motor6">
-            <mechanicalReduction>1</mechanicalReduction>
-        </actuator>
-    </transmission>
-    <!-- <transmission name="${prefix}tran7">
-        <type>transmission_interface/SimpleTransmission</type>
-        <joint name="${prefix}vacuum_joint">
-            <hardwareInterface>EffortJointInterface</hardwareInterface>
-        </joint>
-        <actuator name="motor6">
-            <hardwareInterface>EffortJointInterface</hardwareInterface>
-            <mechanicalReduction>1</mechanicalReduction>
-        </actuator>
-    </transmission> -->
-    <!-- Gazebo-specific link properties -->
-    <gazebo reference="${irb120_ns}base_link">
-        <material>Gazebo/Orange</material>
-        <turnGravityOff>true</turnGravityOff>
-    </gazebo>
-    <gazebo reference="${irb120_ns}link_1">
-        <material>Gazebo/Orange</material>
-        <turnGravityOff>true</turnGravityOff>
-    </gazebo>
-    <gazebo reference="${irb120_ns}link_2">
-        <material>Gazebo/Orange</material>
-        <turnGravityOff>true</turnGravityOff>
-    </gazebo>
-    <gazebo reference="${irb120_ns}link_3">
-        <material>Gazebo/Orange</material>
-        <turnGravityOff>true</turnGravityOff>
-    </gazebo>
-    <gazebo reference="${irb120_ns}link_4">
-        <material>Gazebo/Orange</material>
-        <turnGravityOff>true</turnGravityOff>
-    </gazebo>
-    <gazebo reference="${irb120_ns}link_5">
-        <material>Gazebo/Orange</material>
-        <turnGravityOff>true</turnGravityOff>
-    </gazebo>
-    <gazebo reference="${irb120_ns}link_6">
-        <material>Gazebo/Black</material>
-        <turnGravityOff>true</turnGravityOff>
-    </gazebo>
+<?xml version="1.0"?>
+<robot xmlns:xacro="http://ros.org/wiki/xacro">
+  <xacro:include filename="$(find abb_resources)/urdf/common_materials.xacro"/>
+  <xacro:macro name="abb_irb120" params="prefix">
+    <!-- link list -->
+    <link name="${prefix}base_link">
+      <inertial>
+        <mass value="6.215"/>
+        <origin xyz="-0.04204 8.01E-05 0.07964" rpy="0 0 0"/>
+        <inertia ixx="0.0247272" ixy="-8.0784E-05" ixz="0.00130902" iyy="0.0491285" iyz="-8.0419E-06" izz="0.0472376"/>
+      </inertial>
+      <visual>
+        <origin xyz="0 0 0" rpy="0 0 0"/>
+        <geometry>
+          <mesh filename="package://irb120_description/meshes/visual/base_link.stl"/>
+        </geometry>
+        <xacro:material_abb_white />
+      </visual>
+      <collision>
+        <origin xyz="0 0 0" rpy="0 0 0"/>
+        <geometry>
+          <mesh filename="package://irb120_description/meshes/collision/base_link.stl"/>
+        </geometry>
+        <xacro:material_abb_yellow />
+      </collision>
+    </link>
+    <link name="${prefix}link_1">
+      <inertial>
+        <mass value="3.067" />
+        <origin xyz="9.77E-05 -0.00012 0.23841" rpy="0 0 0"/>
+        <inertia ixx="0.0142175" ixy="-1.28579E-05" ixz="-2.31364E-05" iyy="0.0144041" iyz="1.93404E-05" izz="0.0104533"/>
+      </inertial>
+      <visual>
+        <origin xyz="0 0 0" rpy="0 0 0"/>
+        <geometry>
+          <mesh filename="package://irb120_description/meshes/visual/link_1.stl"/>
+        </geometry>
+        <xacro:material_abb_white />
+      </visual>
+      <collision>
+        <origin xyz="0 0 0" rpy="0 0 0"/>
+        <geometry>
+          <mesh filename="package://irb120_description/meshes/collision/link_1.stl"/>
+        </geometry>
+        <xacro:material_abb_yellow />
+      </collision>
+    </link>
+    <link name="${prefix}link_2">
+      <inertial>
+        <mass value="3.909"/>
+        <origin xyz="0.00078 -0.00212 0.10124" rpy="0 0 0"/>
+        <inertia ixx="0.0603111" ixy="9.83431E-06" ixz="5.72407E-05" iyy="0.041569" iyz="-0.00050497" izz="0.0259548"/>
+      </inertial>
+      <visual>
+        <origin xyz="0 0 0" rpy="0 0 0"/>
+        <geometry>
+          <mesh filename="package://irb120_description/meshes/visual/link_2.stl"/>
+        </geometry>
+        <xacro:material_abb_white />
+      </visual>
+      <collision>
+        <origin xyz="0 0 0" rpy="0 0 0"/>
+        <geometry>
+          <mesh filename="package://irb120_description/meshes/collision/link_2.stl"/>
+        </geometry>
+        <xacro:material_abb_yellow />
+      </collision>
+    </link>
+    <link name="${prefix}link_3">
+      <inertial>
+        <mass value="2.944"/>
+        <origin xyz="0.02281 0.00106 0.05791" rpy="0 0 0"/>
+        <inertia ixx="0.00835606" ixy="-8.01545E-05" ixz="0.00142884" iyy="0.016713" iyz="-0.000182227" izz="0.0126984"/>
+      </inertial>
+      <visual>
+        <origin xyz="0 0 0" rpy="0 0 0"/>
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
Commit message: description

File: irb120_description/urdf/irb120.xacro (robot description, xacro)
@@ -197,5 +197,6 @@
       <parent link="${prefix}link_5"/>
       <child link="${prefix}link_6"/>
-      <limit effort="0" lower="-6.98132" upper="6.98132" velocity="7.33038"/>
+      <limit effort="0" lower="-3.98132" upper="3.98132" velocity="7.33038"/>
+      <!-- <limit effort="0" lower="-6.98132" upper="6.98132" velocity="7.33038"/> -->
       <axis xyz="1 0 0"/>
       <dynamics damping="0.0" friction="0.0"/>
